Commit message: change origin

File: robot.urdf (robot description, URDF)
Before this commit: robot dash_urdf, 19 links, 18 joints
Joints:
- joint l_ankle_pitch: origin xyz=1.38778e-17 -0.28 0.0573813 rpy=3.14159 1.0373e-16 -1.09286e-16 -> xyz=1.38778e-17 -0.28 0.0573813 rpy=3.14159 1.0373e-16 -1.0932e-16
- joint l_elbow_pitch: origin xyz=1.2039e-15 0.023275 -0.2025 rpy=-1.5708 -2.71149e-17 -3.14159 -> xyz=2.16493e-15 0.023275 -0.2025 rpy=-1.5708 -2.71149e-17 -3.14159
- joint l_hip_yaw: origin xyz=-0.0484277 0.171044 -0.116218 rpy=0.436097 0.0148252 -0.0318004 -> xyz=0.000796034 0.0747464 0.000543785 rpy=0.436097 0.0148252 -0.0318004
- joint l_knee_pitch: origin xyz=0.114051 -0.255719 -0.0768 rpy=5.02142e-16 -1.14985e-16 0.419523 -> xyz=0.114051 -0.255719 -0.0768 rpy=6.99142e-16 3.66642e-16 0.419523
- joint l_shoulder_pitch: origin xyz=-0.0284277 0.207997 0.183239 rpy=1.5708 1.91569e-13 2.26409e-15 -> xyz=0.020796 0.1117 0.3 rpy=1.5708 1.95566e-13 4.37509e-14
- joint l_shoulder_roll: origin xyz=-0.0505 -7.16094e-15 -0.0713 rpy=1.52918e-13 -1.5708 0 -> xyz=-0.0505 -8.65974e-15 -0.0713 rpy=1.82506e-13 -1.5708 0
- joint r_ankle_pitch: origin xyz=0 0.28 0.0573813 rpy=3.14159 -3.39931e-15 1.45618e-14 -> xyz=6.93889e-18 0.28 0.0573813 rpy=3.14159 -3.39931e-15 1.45687e-14
- joint r_elbow_pitch: origin xyz=-1.69309e-15 -0.023275 -0.2025 rpy=1.5708 2.31682e-16 -3.14159 -> xyz=-2.67147e-15 -0.023275 -0.2025 rpy=1.5708 2.31682e-16 -3.14159
- joint r_hip_yaw: origin xyz=-0.0484277 0.0215507 -0.116218 rpy=-0.436097 0.0148252 0.0318004 -> xyz=0.000796034 -0.0747464 0.000543785 rpy=-0.436097 0.0148252 0.0318004
- joint r_knee_pitch: origin xyz=0.114051 0.255719 -0.0768 rpy=4.25568e-16 -3.2166e-15 -0.419523 -> xyz=0.114051 0.255719 -0.0768 rpy=4.15811e-16 -3.04566e-15 -0.419523
- joint r_shoulder_pitch: origin xyz=-0.0284277 -0.0154028 0.183239 rpy=-1.5708 1.87628e-13 -5.84474e-16 -> xyz=0.020796 -0.1117 0.3 rpy=-1.5708 1.9168e-13 4.09023e-14
- joint r_shoulder_roll: origin xyz=-0.0554 7.82707e-15 -0.0713 rpy=-3.14159 1.5708 0 -> xyz=-0.0554 9.60343e-15 -0.0713 rpy=-3.14159 1.5708 0

Commit message: upload a clean urdf

File: robot.urdf (robot description, URDF)
Before this commit: robot dash_urdf, 19 links, 18 joints
Links:
- link l_dist_hip: geometry collision mesh filename=package://assets/L_dist_hip.stl; visual mesh filename=package://assets/L_dist_hip.stl
- link l_dist_shoulder: geometry collision mesh filename=package://assets/L_dist_shoulder.stl; visual mesh filename=package://assets/L_dist_shoulder.stl
- link l_foot: geometry collision mesh filename=package://assets/L_foot.stl; visual mesh filename=package://assets/L_foot.stl
- link l_hip: geometry collision mesh filename=package://assets/L_hip.stl; visual mesh filename=package://assets/L_hip.stl
- link l_lower_arm: geometry collision mesh filename=package://assets/L_lower_arm.stl; visual mesh filename=package://assets/L_lower_arm.stl
- link l_lower_leg: geometry collision mesh filename=package://assets/L_lower_leg.stl; visual mesh filename=package://assets/L_lower_leg.stl
- link l_prox_shoulder: geometry collision mesh filename=package://assets/L_prox_shoulder.stl; visual mesh filename=package://assets/L_prox_shoulder.stl
- link l_upper_arm: geometry collision mesh filename=package://assets/L_upper_arm.stl; visual mesh filename=package://assets/L_upper_arm.stl
- link l_upper_leg: mass 2.55931 -> 2.55930642; geometry collision mesh filename=package://assets/L_upper_leg.stl; visual mesh filename=package://assets/L_upper_leg.stl
- link r_dist_hip: mass 1.80155 -> 1.80153; geometry collision mesh filename=package://assets/R_dist_hip.stl; visual mesh filename=package://assets/R_dist_hip.stl
- link r_dist_shoulder: geometry collision mesh filename=package://assets/R_dist_shoulder.stl; visual mesh filename=package://assets/R_dist_shoulder.stl
- link r_foot: mass 0.283056 -> 0.28305631; geometry collision mesh filename=package://assets/R_foot.stl; visual mesh filename=package://assets/R_foot.stl
- link r_hip: geometry collision mesh filename=package://assets/R_hip.stl; visual mesh filename=package://assets/R_hip.stl
- link r_lower_arm: geometry collision mesh filename=package://assets/R_lower_arm.stl; visual mesh filename=package://assets/R_lower_arm.stl
- link r_lower_leg: geometry collision mesh filename=package://assets/R_lower_leg.stl; visual mesh filename=package://assets/R_lower_leg.stl
- link r_prox_shoulder: geometry collision mesh filename=package://assets/R_prox_shoulder.stl; visual mesh filename=package://assets/R_prox_shoulder.stl
- link r_upper_arm: geometry collision mesh filename=package://assets/R_upper_arm.stl; visual mesh filename=package://assets/R_upper_arm.stl
- link r_upper_leg: mass 2.55931 -> 2.55930636; geometry collision mesh filename=package://assets/R_upper_leg.stl; visual mesh filename=package://assets/R_upper_leg.stl
- link torso: geometry collision mesh filename=package://assets/Torso.stl; visual mesh filename=package://assets/Torso.stl
Joints:
- joint l_ankle_pitch: axis 0 0 1 -> 0 1 0; origin xyz=1.38778e-17 -0.28 0.0573813 rpy=3.14159 1.0373e-16 -1.0932e-16 -> xyz=0 0.00034598 -0.28000000 rpy=0 0 0
- joint l_elbow_pitch: axis 0 0 1 -> 0 1 0; origin xyz=2.16493e-15 0.023275 -0.2025 rpy=-1.5708 -2.71149e-17 -3.14159 -> xyz=0 0.02377500 -0.20250000 rpy=0 -0.5 0
- joint l_hip_pitch: axis 0 0 1 -> 0 1 0; origin xyz=-0.000592305 -0.0052668 -0.0953 rpy=1.68279 1.5708 0 -> xyz=0.09530000 -0.00530000 0.00000000 rpy=0 -0.329548199892 0
- joint l_hip_roll: axis 0 0 1 -> 1 0 0; origin xyz=-0.0527293 -0.00277237 -0.081917 rpy=-1.01258 -0.918792 0.986213 -> xyz=-0.05273 -0.00277237 -0.08191703 rpy=-0.436332 0.329548199892 -0.1238480401
- joint l_hip_yaw: origin xyz=0.000796034 0.0747464 0.000543785 rpy=0.436097 0.0148252 -0.0318004 -> xyz=0.00079603 0.0747464 0.000544 rpy=0.43633  0.00000000  0.00000000
- joint l_knee_pitch: axis 0 0 1 -> 0 1 0; origin xyz=0.114051 -0.255719 -0.0768 rpy=6.99142e-16 3.66642e-16 0.419523 -> xyz=0 0.04245000 -0.28000000 rpy=0 0 0
- joint l_shoulder_pitch: axis 0 0 1 -> 0 1 0; origin xyz=0.020796 0.1117 0.3 rpy=1.5708 1.95566e-13 4.37509e-14 -> xyz=0.02079603 0.11200000 0.30000000 rpy=0 0 0
- joint l_shoulder_roll: axis 0 0 1 -> 1 0 0; origin xyz=-0.0505 -8.65974e-15 -0.0713 rpy=1.82506e-13 -1.5708 0 -> xyz=-0.05000000 0.07130000 0 rpy=0 0 0
- joint l_shoulder_yaw: origin xyz=-0.012 0.0025 -0.0605 rpy=-1.5708 1.5708 0 -> xyz=0.06050000 0.01200000 0.00200000 rpy=0 0 0
- joint r_ankle_pitch: axis 0 0 1 -> 0 1 0; origin xyz=6.93889e-18 0.28 0.0573813 rpy=3.14159 -3.39931e-15 1.45687e-14 -> xyz=0 0.00034598 -0.28000000 rpy=0 0 0
- joint r_elbow_pitch: axis 0 0 1 -> 0 1 0; origin xyz=-2.67147e-15 -0.023275 -0.2025 rpy=1.5708 2.31682e-16 -3.14159 -> xyz=0 -0.02377500 -0.20250000 rpy=0 -0.5 0
- joint r_hip_pitch: axis 0 0 1 -> 0 1 0; origin xyz=0.000791025 0.00524064 -0.0953 rpy=-1.42099 1.5708 0 -> xyz=0.09530000 0.00530000 0.00000000 rpy=0 -0.329548199892 0
- joint r_hip_roll: axis 0 0 1 -> 1 0 0; origin xyz=-0.0527293 0.00277237 -0.081917 rpy=0.736507 -1.12205 -0.66471 -> xyz=-0.0527293 0.00277237 -0.08191703 rpy=0.436332 0.329548199892 0.1238480401
- joint r_hip_yaw: origin xyz=0.000796034 -0.0747464 0.000543785 rpy=-0.436097 0.0148252 0.0318004 -> xyz=0.00079603 -0.0747464 0.000544 rpy=-0.43633  0.00000000  0.00000000
- joint r_knee_pitch: axis 0 0 1 -> 0 1 0; origin xyz=0.114051 0.255719 -0.0768 rpy=4.15811e-16 -3.04566e-15 -0.419523 -> xyz=0.0 -0.04245000 -0.28000000 rpy=0 0 0
- joint r_shoulder_pitch: axis 0 0 1 -> 0 1 0; origin xyz=0.020796 -0.1117 0.3 rpy=-1.5708 1.9168e-13 4.09023e-14 -> xyz=0.02079603 -0.11170000 0.30000000 rpy=0 0 0
- joint r_shoulder_roll: axis 0 0 1 -> 1 0 0; origin xyz=-0.0554 9.60343e-15 -0.0713 rpy=-3.14159 1.5708 0 -> xyz=-0.05000000 -0.07130000 0 rpy=0 0 0
- joint r_shoulder_yaw: origin xyz=0.012 0.0025 -0.0605 rpy=-1.5708 1.5708 0 -> xyz=0.06050000 -0.01200000 0.00200000 rpy=0 0 0
